Commit message: update moveit_config

File: phantomx_reactor_arm_description_v2/urdf/phantomx_reactor_arm_no_wrist.urdf.xacro (robot description, xacro)
@@ -12,6 +12,6 @@
   <xacro:property name="wrist_roll_upper_limit" value="${PI}"/>
   <xacro:property name="wrist_roll_lower_limit" value="-${PI}"/>
-  <xacro:property name="gripper_joint_upper_limit" value="0.0"/>
-  <xacro:property name="gripper_joint_lower_limit" value="0.03"/>
+  <xacro:property name="gripper_joint_upper_limit" value="0.03"/>
+  <xacro:property name="gripper_joint_lower_limit" value="0.001"/>
   <xacro:macro name="phantomx_reactor_arm_no_wrist" params="parent prefix *origin">
       <!-- ARM BASE JOINT -->

Commit message: xacro correction

File: phantomx_reactor_arm_description_v2/urdf/phantomx_reactor_arm_no_wrist.urdf.xacro (robot description, xacro)
@@ -10,6 +10,4 @@
   <xacro:property name="wrist_pitch_upper_limit" value="1.9"/>
   <xacro:property name="wrist_pitch_lower_limit" value="-1.7"/>
-  <xacro:property name="wrist_roll_upper_limit" value="${PI}"/>
-  <xacro:property name="wrist_roll_lower_limit" value="-${PI}"/>
   <xacro:property name="gripper_joint_upper_limit" value="0.03"/>
   <xacro:property name="gripper_joint_lower_limit" value="0.001"/>
